Commit message: update

File: jackal_setup/jackal/jackal_description/urdf/accessories.urdf.xacro (robot description, xacro)
@@ -18,4 +18,5 @@
   <xacro:include filename="$(find jackal_description)/urdf/accessories/sick_lms1xx_inverted_mount.urdf.xacro" />
   <xacro:include filename="$(find jackal_description)/urdf/accessories/sick_lms1xx_upright_mount.urdf.xacro" />
+  <xacro:include filename="$(find jackal_description)/urdf/accessories/hokuyo_utm30.urdf.xacro" />
   <xacro:include filename="$(find jackal_description)/urdf/accessories/hokuyo_ust10.urdf.xacro" />
   <xacro:include filename="$(find jackal_description)/urdf/accessories/vlp16_mount.urdf.xacro" />
@@ -25,14 +26,9 @@
     optional microstrain IMU's will be added to another frame, by default, "microstrain_link".
   -->
-  <xacro:property name="microstrain_enable" value="$(optenv JACKAL_GX5_IMU 0)"/>
-  <xacro:property name="microstrain_enable" value="$(optenv JACKAL_IMU_MICROSTRAIN ${microstrain_enable})" lazy_eval="false"/>
-  <xacro:if value="${microstrain_enable}">
+  <xacro:if value="$(optenv JACKAL_IMU_MICROSTRAIN 0)">
     <xacro:property name="frame"  value="$(optenv JACKAL_IMU_MICROSTRAIN_LINK microstrain_link)"/>
-    <xacro:property name="parent" value="$(optenv JACKAL_GX5_IMU_PARENT base_link)"/>
-    <xacro:property name="parent" value="$(optenv JACKAL_IMU_MICROSTRAIN_PARENT ${parent})" lazy_eval="false"/>
-    <xacro:property name="xyz"    value="$(optenv JACKAL_GX5_IMU_OFFSET -0.139 0.096 0.100)"/>
-    <xacro:property name="xyz"    value="$(optenv JACKAL_IMU_MICROSTRAIN_OFFSET ${xyz})" lazy_eval="false"/>
-    <xacro:property name="rpy"    value="$(optenv JACKAL_GX5_IMU_RPY ${PI} 0 -${PI/2})"/>
-    <xacro:property name="rpy"    value="$(optenv JACKAL_IMU_MICROSTRAIN_RPY ${rpy})" lazy_eval="false"/>
+    <xacro:property name="parent" value="$(optenv JACKAL_IMU_MICROSTRAIN_PARENT base_link)"/>
+    <xacro:property name="xyz"    value="$(optenv JACKAL_IMU_MICROSTRAIN_OFFSET -0.139 0.096 0.100)"/>
+    <xacro:property name="rpy"    value="$(optenv JACKAL_IMU_MICROSTRAIN_RPY ${PI} 0 -${PI/2})"/>
     <link name="${frame}" />
     <joint name="${frame}_joint" type="fixed">
@@ -47,4 +43,5 @@
     - lms1xx (default) :: SICK LMS1xx
     - ust10            :: Hokuyo UST10
+    - utm30            :: Hokuyo UTM30
   -->
   <!-- Primary 2D Lidar -->
@@ -104,4 +101,10 @@
       </xacro:hokuyo_ust10_mount>
     </xacro:if>
+    <!-- Hokuyo UTM30 -->
+    <xacro:if value="${lidar_model == 'utm30'}">
+      <xacro:hokuyo_utm30_mount topic="${topic}" prefix="${prefix}" parent_link="${parent}">
+        <origin xyz="$(optenv JACKAL_LASER_OFFSET 0 0 0)" rpy="$(optenv JACKAL_LASER_RPY 0 0 0)" />
+      </xacro:hokuyo_utm30_mount>
+    </xacro:if>
   </xacro:if>
   <!-- Secondary 2D Lidar -->
@@ -153,4 +156,10 @@
       </xacro:hokuyo_ust10_mount>
     </xacro:if>
+    <!-- Hokuyo UTM30 -->
+    <xacro:if value="${lidar_model == 'utm30'}">
+      <xacro:hokuyo_utm30_mount topic="${topic}" prefix="${prefix}" parent_link="${parent}">
+        <origin xyz="$(optenv JACKAL_LASER_SECONDARY_OFFSET 0 0 0)" rpy="$(optenv JACKAL_LASER_SECONDARY_RPY 0 0 3.14159)" />
+      </xacro:hokuyo_utm30_mount>
+    </xacro:if>
   </xacro:if>
   <!--
@@ -371,4 +380,18 @@
     </xacro:unless>
   </xacro:if>
+  <!-- BlackflyS Camera -->
+  <xacro:include filename="$(find flir_camera_description)/urdf/flir_blackflys.urdf.xacro"/>
+  <xacro:if value="$(optenv JACKAL_BLACKFLY 0)">
+    <xacro:property name="prefix" value="$(optenv JACKAL_BLACKFLY_PREFIX front_camera)"/>
+    <xacro:property name="parent" value="$(optenv JACKAL_BLACKFLY_PARENT front_mount)"/>
+    <xacro:property name="xyz"    value="$(optenv JACKAL_BLACKFLY_OFFSET 0 0 0)"/>
+    <xacro:property name="rpy"    value="$(optenv JACKAL_BLACKFLY_RPY    0 0 0)"/>
+    <xacro:flir_blackflys frame="${prefix}"/>
+    <joint name="${prefix}_mount_joint" type="fixed">
+      <child link="${prefix}"/>
+      <parent link="${parent}"/>
+      <origin xyz="${xyz}" rpy="${rpy}" />
+    </joint>
+  </xacro:if>
   <!-- Fender Accessories -->
   <xacro:if value="$(optenv JACKAL_FRONT_ACCESSORY_FENDER 0)">

File: jackal_setup/jackal/jackal_description/urdf/accessories/hokuyo_ust10.urdf.xacro (robot description, xacro)
@@ -3,5 +3,5 @@
   <xacro:macro name="hokuyo_ust10_mount" params="prefix topic parent_link min_angle:=-2.35619 max_angle:=2.35619 *origin">
     <xacro:macro name="hokuyo_ust10" params="frame:=laser topic:=scan sample_size:=720 update_rate:=50
-               min_angle:=${min_angle} max_angle:=${max_angle} min_range:=0.1 max_range:=30.0 robot_namespace:=/">
+               min_angle:=-2.35619 max_angle:=2.35619 min_range:=0.1 max_range:=30.0 robot_namespace:=/">
       <link name="${frame}">
         <inertial>

File: jackal_setup/jackal/jackal_description/urdf/jackal.urdf.xacro (robot description, xacro)
@@ -173,8 +173,5 @@
     <child link="rear_fender_link" />
   </joint>
-  <!-- TODO: Make this internal_imu_link or something, and use a mixed-in xacro
-       to supply the joint between it and imu_link. This is important so that imu_link
-       always points to the "active" IMU. When an upgrade IMU is connected, the
-       internal_imu_link should remain, but imu_link should point to the upgrade one. -->
+  <!-- Default Internal IMU Link -->
   <link name="imu_link">
     <inertial>
@@ -188,5 +185,5 @@
     <child link="imu_link" />
   </joint>
-  <!-- TODO: Same note as applies to imu_link -->
+  <!-- Default NAVSAT Link -->
   <link name="navsat_link">
     <visual>
@@ -227,4 +224,12 @@
        default each one to off.-->
   <xacro:include filename="$(find jackal_description)/urdf/accessories.urdf.xacro" />
+  <!-- OutdoorNav -->
+  <xacro:arg name="outdoornav_enabled"       default="$(optenv OUTDOORNAV_ENABLED 0)" />
+  <xacro:arg name="outdoornav_configuration" default="$(optenv OUTDOORNAV_CONFIGURATION standard)" />
+  <!-- OutdoorNav URDF Config -->
+  <xacro:if value="$(arg outdoornav_enabled)">
+    <xacro:include filename="$(find cpr_onav_description)/urdf/outdoornav_description.urdf.xacro" />
+    <xacro:outdoornav_sensors outdoornav_configuration="$(arg outdoornav_configuration)" />
+  </xacro:if>
   <!-- Optional custom includes. -->
   <xacro:include filename="$(optenv JACKAL_URDF_EXTRAS empty.urdf)" />
